File: pcb/project.kicad_sch (KiCad schematic)
At the start: 25 parts, among them J1 USB_C_Receptacle_USB2.0_14P, J12 Conn_01x04, J19 Conn_01x06, J2 Conn_01x03, J20 Conn_01x06, J25 Conn_01x06, J29 Conn_01x06, J3 Conn_01x03, U1 LM1117MP-3.3, U16 TCA9548APWR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

Commit message: Organised files a bit
Parts:
- C5: footprint (none) -> Capacitor_SMD:C_0805_2012Metric_Pad1.18x1.45mm_HandSolder
Changed lines of the file:
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@@
 		(exclude_from_sim no)
 		(in_bom yes)
-		(on_board yes)
+		(on_board no)
 		(in_pos_files yes)
 		(dnp no)
@@
 			)
 		)
-		(property "Footprint" ""
+		(property "Footprint" "Capacitor_SMD:C_0805_2012Metric_Pad1.18x1.45mm_HandSolder"
 			(at 122.8852 114.3 0)
 			(hide yes)
@@
 		(exclude_from_sim no)
 		(in_bom yes)
-		(on_board yes)
-		(in_pos_files yes)
-		(dnp no)
+		(on_board no)
+		(in_pos_files yes)
+		(dnp no)
