File: pcb/backleds.kicad_pcb (KiCad board)
At the start: 2 copper layers, 39.5 x 39.5 mm, 6 parts, among them J3 Conn_01x03

Commit message: Update production
Parts:
- added REF**: MountingHole_2.1mm, MountingHole:MountingHole_2.1mm, F.Cu at (135.6, 101.8)
- added REF**: MountingHole_2.1mm, MountingHole:MountingHole_2.1mm, F.Cu at (123.8, 93.6)
- added REF**: MountingHole_2.1mm, MountingHole:MountingHole_2.1mm, F.Cu at (119.4, 101.8)
Routing:
- net Net-(D10-VSS): track 130.2 -> 131.5 mm
